File: extras/eagle/hcsr04bracket/hcsr04bracket.brd (EAGLE design)
At the start: 30.5 x 30.5 mm, 11 parts, among them J0 J0, J1 J1, J2 J2

Commit message: Update hcsr04bracket.brd to 1.1.0
Moved diagonal mount out to correct position. Fixed floodfill.
Parts:
- moved H2 2.54 mm to (16.5, 11.1)
Routing:
- net T3: track 4.86 -> 7.40 mm
- net E3: track 4.86 -> 7.40 mm
- net VCC: track 44.6 -> 46.2 mm
- added copper zone on layer 1, net GND
- added copper zone on layer 16, net GND
- removed copper zone on layer 1, net VCC
- removed copper zone on layer 16, net VCC
Other:
- board text added: "v1.1.0"
- board text removed: "v1.0.0"
