File: extras/eagle/octosonar-feather/octosonar-feather.sch (EAGLE design)
At the start: 39 parts, among them IC1 PCF8574TW, U1 74HC125, U2 74HC125

Commit message: forgot the brd file
Parts:
- J1, S0, S1, S2, S3, S4, S5, S6, S7: device SparkFun-Connectors:CONN_041X04_NO_SILK -> redhunter:CONN_041X04_NO_SILK
- J2, J3, J4: device SparkFun-Connectors:CONN_021X02_NO_SILK -> redhunter:CONN_021X02_NO_SILK
