File: extras/eagle/octosonar-feather/octosonar-feather.sch (EAGLE design)
At the start: 39 parts, among them IC1 PCF8574TW, U1 74HC125, U2 74HC125

Commit message: Octosonar v3.0.0 prod featherwing design
Parts:
- A0, A1, A2, JP1, JP2, JP3, JP4, JP5, JP6, JP7, JP8, JP9, V1, V2: device jumper:SJ -> redhunter:SJSJ-NOCREAM
- renumbered S0 to 0, S1 to 1, S2 to 2, S3 to 3, S4 to 4, S5 to 5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
Connections:
- net 5V renamed VS
- net GND: no longer J2.2
- net INT: now also J2.2
Other:
- moved on the sheet: J2
